Commit message: Basic Controller

File: vehicle_gazebo/models/em_3905_base.urdf.xacro (robot description, xacro)
@@ -85,4 +85,7 @@
     <color rgba="0 0 0 1"/>
   </material>
+  <material name="imu_mat">
+    <color rgba="0 1 0 1"/>
+  </material>
   <!-- Null inertial element. This is needed to make the model work with
        Gazebo. -->
@@ -178,4 +181,5 @@
       <limit lower="${-wheel_travel / 2}" upper="${wheel_travel / 2}"
              effort="${shock_eff_limit}" velocity="${shock_vel_limit}"/>
+      <!-- <dynamics damping="50.0"/> -->
     </joint>
     <transmission name="${lr_prefix}_${fr_prefix}_shock_trans">
@@ -201,4 +205,5 @@
       <axis xyz="0 0 -1"/>
       <limit effort="${axle_eff_limit}" velocity="${axle_vel_limit}"/>
+      <!-- <dynamics damping="0.5"/> -->
     </joint>
     <transmission name="${lr_prefix}_${fr_prefix}_axle_trans">
@@ -253,4 +258,5 @@
       <limit lower="${-degrees_45}" upper="${degrees_45}"
              effort="${servo_stall_torque}" velocity="${servo_no_load_speed}"/>
+      <!-- <dynamics damping="2.0"/> -->
     </joint>
     <transmission name="${lr_prefix}_steering_trans">
@@ -274,6 +280,5 @@
                  lr_reflect="${lr_reflect}"/>
   </xacro:macro>
-  <!-- base_link must have geometry so that its axes can be displayed in
-       rviz. -->
+  <!-- base_link-->
   <link name="base_link">
     <visual>
@@ -312,4 +317,5 @@
   </gazebo>
   <joint name="base_link_to_chassis" type="fixed">
+    <origin xyz="0 0 0" rpy="0 0 0"/>
     <parent link="base_link"/>
     <child link="chassis"/>
@@ -333,7 +339,5 @@
         <box size="0.02 0.035 0.002"/>
       </geometry>
-      <material name="imu_mat">
-        <color rgba="0 1 0 1"/>
-      </material>
+      <material name="imu_mat"/>
     </visual>
     <inertial>
@@ -348,3 +352,42 @@
     <child link="imu_link" />
   </joint>
+    <ros2_control name="GazeboSystem" type="system">
+    <hardware>
+      <plugin>gz_ros2_control/GazeboSimSystem</plugin>
+    </hardware>
+      <!-- Rear wheels (driven) -->
+    <joint name="left_rear_axle">
+      <command_interface name="velocity"/>
+      <state_interface name="velocity"/>
+      <state_interface name="position"/>
+    </joint>
+    <joint name="right_rear_axle">
+      <command_interface name="velocity"/>
+      <state_interface name="velocity"/>
+      <state_interface name="position"/>
+    </joint>
+    <!-- Steering joints -->
+    <joint name="left_steering_joint">
+      <command_interface name="position"/>
+      <state_interface name="position"/>
+    </joint>
+    <joint name="right_steering_joint">
+      <command_interface name="position"/>
+      <state_interface name="position"/>
+    </joint>
+    <!-- Front wheels (passive, only state) -->
+    <joint name="left_front_axle">
+      <state_interface name="velocity"/>
+      <state_interface name="position"/>
+    </joint>
+    <joint name="right_front_axle">
+      <state_interface name="velocity"/>
+      <state_interface name="position"/>
+    </joint>
+  </ros2_control>
+  <gazebo>
+    <plugin filename="gz_ros2_control-system" name="gz_ros2_control::GazeboSimROS2ControlPlugin">
+      <parameters>$(find vehicle_gazebo)/config/ackermann_drive_controller.yaml</parameters>
+    </plugin>
+  </gazebo>
 </robot>

Commit message: IMU

File: vehicle_gazebo/models/em_3905_base.urdf.xacro (robot description, xacro)
@@ -334,4 +334,9 @@
                     lr_reflect="-1" fr_reflect="-1"/>
   <!-- IMU frame -->
+  <joint name="imu_joint" type="fixed">
+    <origin xyz="0 0 0.02" rpy="0 0 0"/>
+    <parent link="base_link" />
+    <child link="imu_link" />
+  </joint>
   <link name="imu_link">
     <visual>
@@ -347,10 +352,70 @@
     </inertial>
   </link>
-  <joint name="imu_joint" type="fixed">
-    <origin xyz="0 0 0.02" rpy="0 0 0"/>
-    <parent link="base_link" />
-    <child link="imu_link" />
-  </joint>
-    <ros2_control name="GazeboSystem" type="system">
+  <gazebo reference="imu_link">
+    <sensor name="imu" type="imu">
+      <always_on>1</always_on>
+      <update_rate>200</update_rate>
+      <visualize>true</visualize>
+      <topic>imu</topic>
+      <enable_metrics>true</enable_metrics>
+      <gz_frame_id>imu_link</gz_frame_id>
+        <imu>
+            <!-- Set the covariance matrix -->
+            <angular_velocity>
+                <x>
+                <noise type="gaussian">
+                    <mean>0.0</mean>
+                    <stddev>0.0001</stddev>
+                    <bias_mean>0.0</bias_mean>
+                    <bias_stddev>0.0</bias_stddev>
+                </noise>
+                </x>
+                <y>
+                <noise type="gaussian">
+                    <mean>0.0</mean>
+                    <stddev>0.0001</stddev>
+                    <bias_mean>0.0</bias_mean>
+                    <bias_stddev>0.0</bias_stddev>
+                </noise>
+                </y>
+                <z>
+                <noise type="gaussian">
+                    <mean>0.0</mean>
+                    <stddev>0.0001</stddev>
+                    <bias_mean>0.0</bias_mean>
+                    <bias_stddev>0.0</bias_stddev>
+                </noise>
+                </z>
+            </angular_velocity>
+            <linear_acceleration>
+                <x>
+                <noise type="gaussian">
+                    <mean>0.0</mean>
+                    <stddev>0.01</stddev>
+                    <bias_mean>0.0</bias_mean>
+                    <bias_stddev>0.0</bias_stddev>
+                </noise>
+                </x>
+                <y>
+                <noise type="gaussian">
+                    <mean>0.0</mean>
+                    <stddev>0.01</stddev>
+                    <bias_mean>0.0</bias_mean>
+                    <bias_stddev>0.0</bias_stddev>
+                </noise>
+                </y>
+                <z>
+                <noise type="gaussian">
+                    <mean>0.0</mean>
+                    <stddev>0.01</stddev>
+                    <bias_mean>0.0</bias_mean>
+                    <bias_stddev>0.0</bias_stddev>
+                </noise>
+                </z>
+            </linear_acceleration>
+        </imu>
+    </sensor>
+  </gazebo>
+  <ros2_control name="GazeboSystem" type="system">
     <hardware>
       <plugin>gz_ros2_control/GazeboSimSystem</plugin>

Commit message: track_width fix

File: vehicle_gazebo/models/em_3905_base.urdf.xacro (robot description, xacro)
@@ -172,5 +172,5 @@
   <xacro:macro name="shock"
                params="lr_prefix fr_prefix lr_reflect fr_reflect child">
-    <joint name="${lr_prefix}_${fr_prefix}_shock" type="prismatic">
+    <joint name="${lr_prefix}_${fr_prefix}_shock" type="fixed">
       <parent link="chassis"/>
       <child link="${child}"/>
@@ -181,14 +181,6 @@
       <limit lower="${-wheel_travel / 2}" upper="${wheel_travel / 2}"
              effort="${shock_eff_limit}" velocity="${shock_vel_limit}"/>
-      <!-- <dynamics damping="50.0"/> -->
-    </joint>
-    <transmission name="${lr_prefix}_${fr_prefix}_shock_trans">
-      <type>transmission_interface/SimpleTransmission</type>
-      <joint name="${lr_prefix}_${fr_prefix}_shock">
-      </joint>
-      <actuator name="${lr_prefix}_${fr_prefix}_shock_act">
-        <mechanicalReduction>1</mechanicalReduction>
-      </actuator>
-    </transmission>
+      <!--  <dynamics damping="25.0" friction="2.0"/> -->
+    </joint>
   </xacro:macro>
   <!-- The "wheel" macro defines an axle carrier, axle, and wheel. -->
@@ -207,12 +199,4 @@
       <!-- <dynamics damping="0.5"/> -->
     </joint>
-    <transmission name="${lr_prefix}_${fr_prefix}_axle_trans">
-      <type>transmission_interface/SimpleTransmission</type>
-      <joint name="${lr_prefix}_${fr_prefix}_axle">
-      </joint>
-      <actuator name="${lr_prefix}_${fr_prefix}_axle_act">
-        <mechanicalReduction>1</mechanicalReduction>
-      </actuator>
-    </transmission>
     <link name="${lr_prefix}_${fr_prefix}_wheel">
       <visual>
@@ -241,4 +225,6 @@
     <gazebo reference="${lr_prefix}_${fr_prefix}_wheel">
       <material>Gazebo/Black</material>
+      <mu1>1.0</mu1>
+      <mu2>1.0</mu2>
     </gazebo>
   </xacro:macro>
@@ -258,14 +244,6 @@
       <limit lower="${-degrees_45}" upper="${degrees_45}"
              effort="${servo_stall_torque}" velocity="${servo_no_load_speed}"/>
-      <!-- <dynamics damping="2.0"/> -->
-    </joint>
-    <transmission name="${lr_prefix}_steering_trans">
-      <type>transmission_interface/SimpleTransmission</type>
-      <joint name="${lr_prefix}_steering_joint">
-      </joint>
-      <actuator name="${lr_prefix}_steering_act">
-        <mechanicalReduction>1</mechanicalReduction>
-      </actuator>
-    </transmission>
+      <!-- <dynamics damping="0.2"/> -->
+    </joint>
     <xacro:wheel lr_prefix="${lr_prefix}" fr_prefix="${fr_prefix}"
                  lr_reflect="${lr_reflect}"/>

Commit message: Full_Manual

File: vehicle_gazebo/models/em_3905_base.urdf.xacro (robot description, xacro)
@@ -74,5 +74,5 @@
        6 V. servo_stall_torque is measured in N m. servo_no_load_speed is
        measured in rad/s. -->
-  <xacro:property name="servo_stall_torque" value="0.5649"/>
+  <xacro:property name="servo_stall_torque" value="3.4"/>
   <xacro:property name="servo_no_load_speed" value="4.553"/>
   <material name="battery_mat">
@@ -244,5 +244,5 @@
       <limit lower="${-degrees_45}" upper="${degrees_45}"
              effort="${servo_stall_torque}" velocity="${servo_no_load_speed}"/>
-      <!-- <dynamics damping="0.2"/> -->
+      <!-- <dynamics damping="0.5" friction="0.01"/> -->
     </joint>
     <xacro:wheel lr_prefix="${lr_prefix}" fr_prefix="${fr_prefix}"

Commit message: odometry fix

File: vehicle_gazebo/models/em_3905_base.urdf.xacro (robot description, xacro)
@@ -39,6 +39,6 @@
   <xacro:property name="hub_dia" value="0.09652"/>
   <xacro:property name="tire_dia" value="0.14605"/>
-  <xacro:property name="tire_width" value="0.0889"/>
-  <xacro:property name="hex_hub_depth" value="0.01445"/>
+  <xacro:property name="tire_width" value="0.01"/>
+  <xacro:property name="hex_hub_depth" value="${tire_width / 2 - axle_length}"/>
   <xacro:property name="wheel_mass" value="0.29"/>
   <!-- hex_hub_dist is the distance between left and right hex hubs when
@@ -218,4 +218,12 @@
           <cylinder radius="${tire_dia / 2}" length="${tire_width}"/>
         </geometry>
+        <surface>
+          <friction>
+            <ode>
+              <mu>50.0</mu>
+              <mu2>50.0</mu2>
+            </ode>
+          </friction>
+        </surface>
       </collision>
       <xacro:thick_walled_tube_inertial
@@ -227,4 +235,12 @@
       <mu1>1.0</mu1>
       <mu2>1.0</mu2>
+      <surface>
+        <friction>
+          <ode>
+            <mu>50.0</mu>
+            <mu2>50.0</mu2>
+          </ode>
+        </friction>
+      </surface>
     </gazebo>
   </xacro:macro>
@@ -295,5 +311,5 @@
   </gazebo>
   <joint name="base_link_to_chassis" type="fixed">
-    <origin xyz="0 0 0" rpy="0 0 0"/>
+    <origin xyz="${wheelbase / 2} 0 0" rpy="0 0 0"/>
     <parent link="base_link"/>
     <child link="chassis"/>
@@ -313,5 +329,5 @@
   <!-- IMU frame -->
   <joint name="imu_joint" type="fixed">
-    <origin xyz="0 0 0.02" rpy="0 0 0"/>
+    <origin xyz="${wheelbase / 2} 0 0.02" rpy="0 0 0"/>
     <parent link="base_link" />
     <child link="imu_link" />

Commit message: odom functional

File: vehicle_gazebo/models/em_3905_base.urdf.xacro (robot description, xacro)
@@ -39,6 +39,6 @@
   <xacro:property name="hub_dia" value="0.09652"/>
   <xacro:property name="tire_dia" value="0.14605"/>
-  <xacro:property name="tire_width" value="0.0889"/>
-  <xacro:property name="hex_hub_depth" value="0.01445"/>
+  <xacro:property name="tire_width" value="0.01"/>
+  <xacro:property name="hex_hub_depth" value="${tire_width / 2 - axle_length}"/>
   <xacro:property name="wheel_mass" value="0.29"/>
   <!-- hex_hub_dist is the distance between left and right hex hubs when
@@ -74,5 +74,5 @@
        6 V. servo_stall_torque is measured in N m. servo_no_load_speed is
        measured in rad/s. -->
-  <xacro:property name="servo_stall_torque" value="0.5649"/>
+  <xacro:property name="servo_stall_torque" value="3.4"/>
   <xacro:property name="servo_no_load_speed" value="4.553"/>
   <material name="battery_mat">
@@ -244,5 +244,5 @@
       <limit lower="${-degrees_45}" upper="${degrees_45}"
              effort="${servo_stall_torque}" velocity="${servo_no_load_speed}"/>
-      <!-- <dynamics damping="0.2"/> -->
+      <!-- <dynamics damping="0.5" friction="0.01"/> -->
     </joint>
     <xacro:wheel lr_prefix="${lr_prefix}" fr_prefix="${fr_prefix}"
@@ -295,5 +295,5 @@
   </gazebo>
   <joint name="base_link_to_chassis" type="fixed">
-    <origin xyz="0 0 0" rpy="0 0 0"/>
+    <origin xyz="${wheelbase / 2} 0 0" rpy="0 0 0"/>
     <parent link="base_link"/>
     <child link="chassis"/>
@@ -313,5 +313,5 @@
   <!-- IMU frame -->
   <joint name="imu_joint" type="fixed">
-    <origin xyz="0 0 0.02" rpy="0 0 0"/>
+    <origin xyz="${wheelbase / 2} 0 0.02" rpy="0 0 0"/>
     <parent link="base_link" />
     <child link="imu_link" />

Commit message: mag_v1

File: vehicle_gazebo/models/em_3905_base.urdf.xacro (robot description, xacro)
@@ -39,5 +39,5 @@
   <xacro:property name="hub_dia" value="0.09652"/>
   <xacro:property name="tire_dia" value="0.14605"/>
-  <xacro:property name="tire_width" value="0.01"/>
+  <xacro:property name="tire_width" value="0.05"/>
   <xacro:property name="hex_hub_depth" value="${tire_width / 2 - axle_length}"/>
   <xacro:property name="wheel_mass" value="0.29"/>
@@ -395,4 +395,41 @@
     </sensor>
   </gazebo>
+  <!-- Magnetometer sensor -->
+  <gazebo reference="imu_link">
+    <sensor name="magnetometer" type="magnetometer">
+      <always_on>true</always_on>
+      <update_rate>50</update_rate>
+      <visualize>false</visualize>
+      <topic>magnetometer</topic>
+      <enable_metrics>true</enable_metrics>
+      <gz_frame_id>imu_link</gz_frame_id>
+      <magnetometer>
+        <x>
+          <noise type="gaussian">
+            <mean>0.0</mean>
+            <stddev>0.000000080</stddev>
+            <bias_mean>0.0</bias_mean>
+            <bias_stddev>0.000000400</bias_stddev>
+          </noise>
+        </x>
+        <y>
+          <noise type="gaussian">
+            <mean>0.0</mean>
+            <stddev>0.000000080</stddev>
+            <bias_mean>0.0</bias_mean>
+            <bias_stddev>0.000000400</bias_stddev>
+          </noise>
+        </y>
+        <z>
+          <noise type="gaussian">
+            <mean>0.0</mean>
+            <stddev>0.000000080</stddev>
+            <bias_mean>0.0</bias_mean>
+            <bias_stddev>0.000000400</bias_stddev>
+          </noise>
+        </z>
+      </magnetometer>
+    </sensor>
+  </gazebo>
   <!-- Groud Truth Pose -->
   <gazebo>

Commit message: cov_correction

File: vehicle_gazebo/models/em_3905_base.urdf.xacro (robot description, xacro)
@@ -39,5 +39,5 @@
   <xacro:property name="hub_dia" value="0.09652"/>
   <xacro:property name="tire_dia" value="0.14605"/>
-  <xacro:property name="tire_width" value="0.05"/>
+  <xacro:property name="tire_width" value="0.01"/>
   <xacro:property name="hex_hub_depth" value="${tire_width / 2 - axle_length}"/>
   <xacro:property name="wheel_mass" value="0.29"/>
@@ -405,29 +405,23 @@
       <gz_frame_id>imu_link</gz_frame_id>
       <magnetometer>
-        <x>
-          <noise type="gaussian">
-            <mean>0.0</mean>
-            <stddev>0.000000080</stddev>
-            <bias_mean>0.0</bias_mean>
-            <bias_stddev>0.000000400</bias_stddev>
-          </noise>
-        </x>
-        <y>
-          <noise type="gaussian">
-            <mean>0.0</mean>
-            <stddev>0.000000080</stddev>
-            <bias_mean>0.0</bias_mean>
-            <bias_stddev>0.000000400</bias_stddev>
-          </noise>
-        </y>
-        <z>
-          <noise type="gaussian">
-            <mean>0.0</mean>
-            <stddev>0.000000080</stddev>
-            <bias_mean>0.0</bias_mean>
-            <bias_stddev>0.000000400</bias_stddev>
-          </noise>
-        </z>
-      </magnetometer>
+          <x>
+            <noise type="gaussian">
+              <mean>0.000000080</mean>
+              <bias_mean>0.000000400</bias_mean>
+            </noise>
+          </x>
+          <y>
+            <noise type="gaussian">
+              <mean>0.000000080</mean>
+              <bias_mean>0.000000400</bias_mean>
+            </noise>
+          </y>
+          <z>
+            <noise type="gaussian">
+              <mean>0.000000080</mean>
+              <bias_mean>0.000000400</bias_mean>
+            </noise>
+          </z>
+        </magnetometer>
     </sensor>
   </gazebo>

Commit message: GPS working

File: vehicle_gazebo/models/em_3905_base.urdf.xacro (robot description, xacro)
@@ -408,5 +408,4 @@
             <noise type="gaussian">
               <mean>0.000000080</mean>
-              <!-- <bias_mean>0.000000400</bias_mean> -->
             </noise>
           </x>
@@ -414,5 +413,4 @@
             <noise type="gaussian">
               <mean>0.000000080</mean>
-              <!-- <bias_mean>0.000000400</bias_mean> -->
             </noise>
           </y>
@@ -420,8 +418,69 @@
             <noise type="gaussian">
               <mean>0.000000080</mean>
-              <!-- <bias_mean>0.000000400</bias_mean> -->
             </noise>
           </z>
         </magnetometer>
+    </sensor>
+  </gazebo>
+  <!-- GPS/GNSS Sensor -->
+  <joint name="gps_joint" type="fixed">
+    <origin xyz="0.0 0.0 0.1" rpy="0 0 0"/>
+    <parent link="base_link"/>
+    <child link="gps_link"/>
+  </joint>
+  <link name="gps_link">
+    <visual>
+      <geometry>
+        <cylinder radius="0.02" length="0.05"/>
+      </geometry>
+      <material name="gps_mat">
+        <color rgba="1 1 0 1"/>
+      </material>
+    </visual>
+    <inertial>
+      <mass value="0.01"/>
+      <origin xyz="0 0 0"/>
+      <inertia ixx="0.0001" ixy="0.0" ixz="0.0"
+               iyy="0.0001" iyz="0.0" izz="0.0001"/>
+    </inertial>
+  </link>
+  <gazebo reference="gps_link">
+    <sensor name="gps" type="navsat">
+      <always_on>true</always_on>
+      <update_rate>10</update_rate>
+      <topic>gps/fix</topic>
+      <gz_frame_id>gps_link</gz_frame_id>
+      <navsat>
+        <position_sensing>
+          <horizontal>
+            <noise type="gaussian">
+              <mean>0.0</mean>
+              <stddev>0.00000018</stddev>  <!-- ±2cm horizontal -->
+              <bias_mean>0.0</bias_mean>
+            </noise>
+          </horizontal>
+          <vertical>
+            <noise type="gaussian">
+              <mean>0.0</mean>
+              <stddev>0.05</stddev>  <!-- ±5cm vertical -->
+              <bias_mean>0.0</bias_mean>
+            </noise>
+          </vertical>
+        </position_sensing>
+        <velocity_sensing>
+          <horizontal>
+            <noise type="gaussian">
+              <mean>0.0</mean>
+              <stddev>0.01</stddev>  <!-- ±1 cm/s -->
+            </noise>
+          </horizontal>
+          <vertical>
+            <noise type="gaussian">
+              <mean>0.0</mean>
+              <stddev>0.02</stddev>  <!-- ±2 cm/s -->
+            </noise>
+          </vertical>
+        </velocity_sensing>
+      </navsat>
     </sensor>
   </gazebo>
