Commit message: potholes_v1

File: vehicle_gazebo/models/prius.urdf.xacro (robot description, xacro)
@@ -37,4 +37,5 @@
   <material name="imu_mat">    <color rgba="0.0 1.0 0.0 1"/></material>
   <material name="gps_mat">    <color rgba="1.0 1.0 1.0 1"/></material>
+  <material name="cam_mat">    <color rgba="0.6 0.0 0.0 1"/></material>
   <!-- ============================================================
        NULL INERTIA MACRO (for kinematic links)
@@ -388,4 +389,47 @@
   </gazebo>
   <!-- ============================================================
+     SEGMENTATION CAMERA (Dashcam position)
+     ============================================================ -->
+<joint name="seg_camera_joint" type="fixed">
+  <origin xyz="0 -0.45 1.28" rpy="0 0.087 -1.5708"/>  <!-- pitch 5° lookdown -->
+  <parent link="chassis"/>
+  <child link="seg_camera_link"/>
+</joint>
+<link name="seg_camera_link">
+  <visual>
+    <geometry>
+      <box size="0.02 0.04 0.03"/>
+    </geometry>
+    <material name="cam_mat"/>
+  </visual>
+  <inertial>
+    <mass value="0.050"/>
+    <origin xyz="0 0 0"/>
+    <inertia ixx="0.0001" ixy="0" ixz="0"
+             iyy="0.0001" iyz="0" izz="0.0001"/>
+  </inertial>
+</link>
+<gazebo reference="seg_camera_link">
+  <sensor name="segmentation_camera" type="segmentation">
+    <topic>segmentation</topic>
+    <camera>
+      <segmentation_type>semantic</segmentation_type>
+      <!-- FOV ~80° -->
+      <horizontal_fov>1.3963</horizontal_fov>
+      <image>
+        <width>1280</width>
+        <height>720</height>
+      </image>
+      <clip>
+        <near>0.5</near>
+        <far>80.0</far>  <!-- 80m -->
+      </clip>
+    </camera>
+    <always_on>1</always_on>
+    <update_rate>30</update_rate>
+    <visualize>true</visualize>
+  </sensor>
+</gazebo>
+  <!-- ============================================================
        GROUND TRUTH ODOMETRY
        ============================================================ -->
